Commit message: Updated URDF and added slam parameters

File: sec_bot_ros2/urdf/URDF.xacro (robot description, xacro)
@@ -5,4 +5,6 @@
 <xacro:include filename="$(find sec_bot_ros2)/urdf/URDF.gazebo" />
 <link name="base_link">
+</link>
+<link name="base_footprint">
 </link>
 <link name="chassis_link">
@@ -106,4 +108,9 @@
   </collision>
 </link>
+<joint name="base_footprint_joint" type="fixed">
+  <parent link="base_link"/>
+  <child link="base_footprint"/>
+  <origin xyz="0 0 0" rpy = "0 0 0"/>
+</joint>
 <joint name="chassis_joint" type="fixed">
   <origin xyz="0 0 0" rpy="0 0 0"/>

Commit message: New Lidar Module

File: sec_bot_ros2/urdf/URDF.xacro (robot description, xacro)
@@ -109,7 +109,7 @@
 </link>
 <joint name="base_footprint_joint" type="fixed">
+  <origin xyz="0 0 0" rpy = "0 0 0"/>
   <parent link="base_link"/>
   <child link="base_footprint"/>
-  <origin xyz="0 0 0" rpy = "0 0 0"/>
 </joint>
 <joint name="chassis_joint" type="fixed">

Commit message: Made bringup easier

File: sec_bot_ros2/urdf/URDF.xacro (robot description, xacro)
@@ -125,5 +125,5 @@
 </joint>
 <joint name="lidar_joint" type="fixed">
-  <origin xyz="0.0 -0.079076 0.100631" rpy="0 0 0"/>
+  <origin xyz="0.0 -0.079076 0.100631" rpy="0 0 1.570796"/>
   <parent link="base_link"/>
   <child link="lidar_link"/>
